Commit message: 수정

File: src/turtlebot3_velodyne/turtlebot3_velodyne_description/urdf/turtlebot3_burger.gazebo.xacro (robot description, xacro)
@@ -91,3 +91,34 @@
     </plugin>
   </gazebo>
+<!-- Camera Gazebo plugin -->
+<gazebo reference="camera_link">
+  <sensor type="camera" name="camera_sensor">
+    <camera>
+      <horizontal_fov>1.3962634</horizontal_fov>
+      <image>
+        <width>800</width>
+        <height>600</height>
+        <format>R8G8B8</format>
+      </image>
+      <clip>
+        <near>0.1</near>
+        <far>300</far>
+      </clip>
+    </camera>
+    <plugin name="camera_controller" filename="libgazebo_ros_camera.so">
+      <alwaysOn>true</alwaysOn>
+      <updateRate>30.0</updateRate>
+      <cameraName>camera</cameraName>
+      <imageTopicName>/camera/rgb/image_raw</imageTopicName>
+      <cameraInfoTopicName>/camera/rgb/camera_info</cameraInfoTopicName>
+      <frameName>camera_link</frameName>
+      <hackBaseline>0.07</hackBaseline>
+      <distortionK1>0.0</distortionK1>
+      <distortionK2>0.0</distortionK2>
+      <distortionK3>0.0</distortionK3>
+      <distortionT1>0.0</distortionT1>
+      <distortionT2>0.0</distortionT2>
+    </plugin>
+  </sensor>
+</gazebo>
 </robot>

File: src/turtlebot3_velodyne/turtlebot3_velodyne_description/urdf/turtlebot3_burger.urdf.xacro (robot description, xacro)
@@ -19,5 +19,4 @@
         <mesh filename="package://turtlebot3_velodyne_description/meshes/bases/burger_base.stl" scale="0.001 0.001 0.001"/>
       </geometry>
-      <material name="light_black"/>
     </visual>
     <collision>
@@ -117,13 +116,52 @@
   </joint>
   <link name="imu_link"/>
-  <xacro:include filename="$(find turtlebot3_velodyne_description)/urdf/VLP-16.urdf.xacro"/>
+  <joint name="scan_joint" type="fixed">
+      <parent link="base_link"/>
+      <child link="base_scan"/>
+      <!-- 센서의 높이와 위치를 조정 -->
+      <origin xyz="0 0 0.1" rpy="0 0 0"/> <!-- z 값을 낮춰 센서가 덜 "붕 뜨도록" 조정 -->
+  </joint>
+  <link name="base_scan">
+      <visual>
+          <origin xyz="0 0 0" rpy="0 0 0"/>
+          <geometry>
+              <box size="0.05 0.05 0.05"/>
+          </geometry>
+          <material name="black"/>
+      </visual>
+  </link>
+</link>
+  <joint name="camera_joint" type="fixed">
+    <origin xyz="0.073 -0.011 0.084" rpy="0 0 0"/>
+    <parent link="base_link"/>
+    <child link="camera_link"/>
+  </joint>
+  <link name="camera_link">
+    <collision>
+      <origin xyz="0.005 0.011 0.013" rpy="0 0 0"/>
+      <geometry>
+        <box size="0.015 0.030 0.027"/>
+      </geometry>
+    </collision>
+  </link>
+  <joint name="camera_rgb_joint" type="fixed">
+    <origin xyz="0.003 0.011 0.009" rpy="0 0 0"/>
+    <parent link="camera_link"/>
+    <child link="camera_rgb_frame"/>
+  </joint>
+  <link name="camera_rgb_frame"/>
+  <joint name="camera_rgb_optical_joint" type="fixed">
+    <origin xyz="0 0 0" rpy="-1.57 0 -1.57"/>
+    <parent link="camera_rgb_frame"/>
+    <child link="camera_rgb_optical_frame"/>
+  </joint>
+  <link name="camera_rgb_optical_frame"/>
+  <!-- <xacro:include filename="$(find turtlebot3_velodyne_description)/urdf/VLP-16.urdf.xacro"/>
   <xacro:VLP-16 parent="base_link" name="velodyne" topic="/velodyne_points" organize_cloud="${organize_cloud}" hz="10" samples="440" gpu="${gpu}">
     <origin xyz="-0.032 0 0.14" rpy="0 0 0" />
-  </xacro:VLP-16>
-  <!-- for HDL-32E
+  </xacro:VLP-16> -->
     <xacro:include filename="$(find turtlebot3_velodyne_description)/urdf/HDL-32E.urdf.xacro"/>
-  <xacro:HDL-32E parent="base_link" name="velodyne2" topic="/velodyne_points2" organize_cloud="${organize_cloud}" hz="10" samples="220" gpu="${gpu}">
+  <xacro:HDL-32E parent="base_scan" name="velodyne2" topic="/velodyne_points2" organize_cloud="${organize_cloud}" hz="10" samples="220" gpu="${gpu}">
     <origin xyz="-0.032 0 0.14" rpy="0 0 0" />
   </xacro:HDL-32E>
-  -->
 </robot>
